File: shawazu-gb-dumper.kicad_pcb (KiCad board)
At the start: 2 copper layers, 70 x 90 mm, 16 parts, among them J1 GB_CART, SW1 VSEL, U1 BOB-12009, U2 BOB-12009, U3 BOB-12009, U4 BOB-12009, U5 BOB-12009, U6 BOB-12009, U7 BOB-12009, U8 Pico

Commit message: new PCB release
Parts:
- moved J1 1.02 mm to (140.0, 46.0)
Routing:
- net D7: track 18.5 -> 21.1 mm
- net A4: track 30.9 -> 28.9 mm
- net A1: track 19.0 -> 20.9 mm
- net GND: track 344.0 -> 345.3 mm
- net D5: track 11.3 -> 12.4 mm
- net PWR: track 219.3 -> 220.4 mm
- net A3: track 13.2 -> 14.3 mm
- net D6: track 17.5 -> 18.5 mm
- net D4: track 10.8 -> 11.9 mm
- net A2: track 14.1 -> 14.9 mm
- net A0: track 20.0 -> 20.6 mm
- net D1: track 9.92 -> 10.5 mm
- net A7: track 25.2 -> 25.8 mm
- net A6: track 25.8 -> 26.4 mm
- net A5: track 27.8 -> 28.5 mm
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Other:
- outline, holes or cut-outs redrawn

Commit message: pcb v2 (actually)
Routing:
- net GND: track 345.3 -> 345.7 mm, vias 3 -> 66
- added copper zone on F.Cu, net GND

Commit message: add more vias because vias are free (this on i actually ordered)
Routing:
- net GND: track 345.7 -> 355.0 mm, vias 66 -> 90

Commit message: rev4
Parts:
- added TP4: ~{CS2}, TestPoint:TestPoint_Pad_D2.0mm, F.Cu at (170.0, 89.5)
- 10 kΩ: renamed from R1
- renumbered PICO_TP4 to TP1
Routing:
- net ~{RST}: track 53.8 -> 57.2 mm
Other:
- board text added: "rev4"
Changed lines of the file:
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@@
 		(descr "Plated Hole as test Point, diameter 4.0mm")
 		(tags "test point plated hole")
-		(property "Reference" "PICO_TP4"
+		(property "Reference" "TP1"
 			(at 2 -3.5 180)
 			(layer "F.SilkS")
@@
 	(footprint "TestPoint:TestPoint_Pad_D2.0mm"
 		(layer "F.Cu")
+		(at 170 89.5)
+		(descr "SMD pad as test Point, diameter 2.0mm")
+		(tags "test point SMD pad")
+		(property "Reference" "TP4"
+			(at 0 -1.998 0)
+			(layer "F.SilkS")
+			(hide yes)
+			(effects
+				(font
+					(size 1 1)
+					(thickness 0.15)
+				)
+			)
+		)
+		(property "Value" "~{CS2}"
+			(at 0 3 0)
+			(layer "F.SilkS")
+			(effects
+				(font
+					(size 1 1)
+					(thickness 0.15)
+				)
+			)
+		)
+		(property "Footprint" "TestPoint:TestPoint_Pad_D2.0mm"
+			(at 0 0 0)
+			(unlocked yes)
+			(layer "F.Fab")
+			(hide yes)
+			(effects
+				(font
+					(size 1.27 1.27)
+				)
+			)
+		)
+		(property "Datasheet" ""
+			(at 0 0 0)
+			(unlocked yes)
+			(layer "F.Fab")
+			(hide yes)
+			(effects
+				(font
+					(size 1.27 1.27)
+				)
+			)
+		)
+		(property "Description" "test point"
+			(at 0 0 0)
+			(unlocked yes)
+			(layer "F.Fab")
+			(hide yes)
+			(effects
+				(font
+					(size 1.27 1.27)
+				)
+			)
+		)
+		(property ki_fp_filters "Pin* Test*")
+		(sheetname "Root")
+		(sheetfile "shawazu-gb-dumper.kicad_sch")
+		(attr exclude_from_pos_files)
+		(fp_circle
+			(center 0 0)
+			(end 0 1.2)
+			(stroke
+				(width 0.12)
+				(type solid)
+			)
+			(fill none)
+			(layer "F.SilkS")
+		)
+		(fp_circle
+			(center 0 0)
+			(end 1.5 0)
+			(stroke
+				(width 0.05)
+				(type solid)
+			)
+			(fill none)
+			(layer "F.CrtYd")
+		)
+		(pad "1" smd circle
+			(at 0 0)
+			(size 2 2)
+			(layers "F.Cu" "F.Mask")
+			(net 28 "~{RST}")
+			(pinfunction "1")
+			(pintype "passive")
+		)
+	)
+	(footprint "TestPoint:TestPoint_Pad_D2.0mm"
+		(layer "F.Cu")
 		(at 114.5 78)
 		(descr "SMD pad as test Point, diameter 2.0mm")
@@
 		(descr "Resistor, Axial_DIN0309 series, Axial, Horizontal, pin pitch=12.7mm, 0.5W = 1/2W, length*diameter=9*3.2mm^2, http://cdn-reichelt.de/documents/datenblatt/B400/1_4W%23YAG.pdf")
 		(tags "Resistor Axial_DIN0309 series Axial Horizontal pin pitch 12.7mm 0.5W = 1/2W length 9mm diameter 3.2mm")
-		(property "Reference" "R1"
-			(at 6.35 -2.72 -90)
+		(property "Reference" "10 kΩ"
+			(at 6.35 -2.72 270)
 			(layer "F.SilkS")
 			(effects
@@
 			(at 6.35 2.72 -90)
 			(layer "F.Fab")
+			(hide yes)
 			(effects
 				(font
@@
 			(layer "F.Fab")
 		)
-		(fp_text user "${REFERENCE}"
-			(at 6.35 0 0)
-			(layer "F.Fab")
-			(effects
-				(font
-					(size 1 1)
-					(thickness 0.15)
-				)
-			)
-		)
 		(pad "1" thru_hole circle
 			(at 0 0 90)
@@
 		)
 	)
+	(gr_text "rev4"
+		(at 161 109 0)
+		(layer "F.SilkS")
+		(effects
+			(font
+				(size 1 1)
+				(thickness 0.1)
+			)
+			(justify bottom)
+		)
+	)
 	(gr_text "GND"
 		(at 115 60 0)
@@
 		(width 0.2)
 		(layer "F.Cu")
+		(net 28)
+	)
+	(segment
+		(start 170 89.5)
+		(end 170 86.15)
+		(width 0.2)
+		(layer "F.Cu")
