File: shawazu-gb-dumper.kicad_sch (KiCad schematic)
At the start: 15 parts, among them J1 GB_CART, SW1 VSEL, U1 BOB-12009, U2 BOB-12009, U3 BOB-12009, U4 BOB-12009, U5 BOB-12009, U6 BOB-12009, U7 BOB-12009, U8 Pico

Commit message: rev4
Parts:
- added TP4: ~{CS2}, TestPoint:TestPoint_Pad_D2.0mm, symbol Connector:TestPoint
Connections:
- net ~{RST}: now also TP4.1
Other:
- moved on the sheet: R1
Changed lines of the file:
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@@
 	)
 	(junction
+		(at 233.68 151.13)
+		(diameter 0)
+		(color 0 0 0 0)
+	)
+	(junction
 		(at 139.7 99.06)
 		(diameter 0)
@@
 	(wire
 		(pts
+			(xy 233.68 151.13) (xy 238.76 151.13)
+		)
+		(stroke
+			(width 0)
+			(type default)
+		)
+	)
+	(wire
+		(pts
 			(xy 66.04 31.75) (xy 69.85 31.75)
 		)
@@
 	(wire
 		(pts
+			(xy 228.6 151.13) (xy 233.68 151.13)
+		)
+		(stroke
+			(width 0)
+			(type default)
+		)
+	)
+	(wire
+		(pts
 			(xy 139.7 62.23) (xy 139.7 64.77)
 		)
@@
 	(global_label "PWR"
 		(shape input)
-		(at 228.6 151.13 180)
+		(at 220.98 151.13 180)
 		(fields_autoplaced yes)
 		(effects
@@
 		)
 		(property "Intersheetrefs" "${INTERSHEET_REFS}"
-			(at 221.6234 151.13 0)
+			(at 214.0034 151.13 0)
 			(effects
 				(font
@@
 	(global_label "~{RST}"
 		(shape input)
-		(at 236.22 151.13 0)
+		(at 238.76 151.13 0)
 		(fields_autoplaced yes)
 		(effects
@@
 		)
 		(property "Intersheetrefs" "${INTERSHEET_REFS}"
-			(at 242.6523 151.13 0)
+			(at 245.1923 151.13 0)
 			(effects
 				(font
@@
 	(symbol
 		(lib_id "Device:R")
-		(at 232.41 151.13 90)
+		(at 224.79 151.13 90)
 		(unit 1)
 		(exclude_from_sim no)
@@
 		(fields_autoplaced yes)
 		(property "Reference" "R1"
-			(at 232.41 144.78 90)
+			(at 224.79 144.78 90)
 			(effects
 				(font
@@
 		)
 		(property "Value" "10K Ω"
-			(at 232.41 147.32 90)
+			(at 224.79 147.32 90)
 			(effects
 				(font
@@
 		)
 		(property "Footprint" "Resistor_THT:R_Axial_DIN0309_L9.0mm_D3.2mm_P12.70mm_Horizontal"
-			(at 232.41 152.908 90)
+			(at 224.79 152.908 90)
 			(effects
 				(font
@@
 		)
 		(property "Datasheet" "~"
-			(at 232.41 151.13 0)
+			(at 224.79 151.13 0)
 			(effects
 				(font
@@
 		)
 		(property "Description" "Resistor"
-			(at 232.41 151.13 0)
+			(at 224.79 151.13 0)
 			(effects
 				(font
@@
 					(unit 1)
 				)
+			)
+		)
+	)
+	(symbol
+		(lib_id "Connector:TestPoint")
+		(at 233.68 151.13 0)
+		(unit 1)
+		(exclude_from_sim no)
+		(in_bom yes)
+		(on_board yes)
+		(dnp no)
+		(property "Reference" "TP4"
+			(at 234.95 145.034 0)
+			(effects
+				(font
+					(size 1.27 1.27)
+				)
+				(justify left)
+			)
+		)
+		(property "Value" "~{CS2}"
+			(at 234.696 147.574 0)
+			(effects
+				(font
+					(size 1.27 1.27)
+				)
+				(justify left)
+			)
+		)
+		(property "Footprint" "TestPoint:TestPoint_Pad_D2.0mm"
+			(at 238.76 151.13 0)
+			(effects
+				(font
+					(size 1.27 1.27)
+				)
+				(hide yes)
+			)
+		)
+		(property "Datasheet" "~"
+			(at 238.76 151.13 0)
+			(effects
+				(font
+					(size 1.27 1.27)
+				)
+				(hide yes)
+			)
+		)
+		(property "Description" "test point"
+			(at 233.68 151.13 0)
+			(effects
+				(font
+					(size 1.27 1.27)
+				)
+				(hide yes)
+			)
+		)
+		(pin "1"
+		)
+		(instances
+			(project "shawazu-gb-dumper"
+				(path "/97e0a329-8697-49bc-b4ba-9c706c6dd8be"
+					(reference "TP4")
+					(unit 1)
+				)
